Commit message: updated conf, no dagana for the exp

File: inail2arm_urdf/config/inail2arm.urdf.xacro (robot description, xacro)
@@ -3,5 +3,5 @@
 <xacro:property name="model_name" value="inail2arm" />
 <xacro:property name="model_version" value="0.1" />
-<xacro:arg name="end_effector" default="dagana_fixed"/> <!-- none, ball, dagana_fixed, dagana -->
+<xacro:arg name="end_effector" default="none"/> <!-- none, ball, dagana_fixed, dagana -->
 <xacro:property name="END_EFFECTOR" value="$(arg end_effector)" />
 <!-- HACK to add standalone dagana plugin and ignore the dagana joint in the libxbot2_gz_joint_server -->

File: inail2arm_urdf/urdf/inail2arm.urdf (robot description, URDF)
Before this commit: robot inail2arm, 21 links, 20 joints
Links:
- removed link dagana_1_bottom_link
- removed link dagana_1_tcp
- removed link dagana_1_top_link
Joints:
- removed joint dagana_1_claw_joint
- removed joint dagana_1_mount_joint
- removed joint dagana_1_tcp_joint
- joint j_tcp_1: origin xyz=0 0 0 rpy=0 0 0 -> xyz=0 0 0 rpy=0. 0. 0.; parent dagana_1_tcp -> arm1_6

File: inail2arm_urdf/urdf/inail2arm_macro.urdf.xacro (robot description, xacro)
@@ -139,23 +139,4 @@
                iyy="${Wrist_2_yy}" iyz="${rot*Wrist_2_yz}" izz="${Wrist_2_zz}" />
          </inertial>
-         <!-- <visual>
-            <origin xyz="0.0 0.0 0.0" rpy="0.0 0.0 0.0" />
-            <geometry>
-               <mesh
-                  filename="package://inail2arm_urdf/meshes/mesh_wrist-pitch.stl"
-                  scale="0.001
-               ${rot*0.001} 0.001" />
-            </geometry>
-            <material name="blue" />
-         </visual>
-         <collision>
-            <origin xyz="0.0 0.0 0.0" rpy="0.0 0.0 0.0" />
-            <geometry>
-               <mesh
-                  filename="package://inail2arm_urdf/meshes/simple/mesh_wrist-pitch.stl"
-                  scale="0.001
-               ${rot*0.001} 0.001" />
-            </geometry>
-         </collision> -->
       </link>
       <!--wrist-pitch -->
