Commit message: debugging launches and xacro to use gazebo and xbot togheter with the fixed arm on the table AND camera position first trial

File: inail2arm_urdf/urdf/inail2arm.urdf (robot description, URDF)
Before this commit: robot inail2arm, 12 links, 11 joints
Links:
- removed link world
Joints:
- removed joint base_joint

File: inail2arm_urdf/urdf/inail2arm.urdf.xacro (robot description, xacro)
@@ -7,4 +7,5 @@
     <xacro:arg name="pitch" default="0"/>
     <xacro:arg name="yaw" default="0"/>
+    <xacro:arg name="parent" default=""/>
     <xacro:include filename="$(find inail2arm_urdf)/config/inail2arm.urdf.xacro" />
     <xacro:include filename="$(find inail2arm_urdf)/urdf/conversions.urdf.xacro" />
@@ -16,7 +17,6 @@
     <xacro:include filename="$(find inail2arm_urdf)/urdf/inertial_properties.urdf.xacro" />
     <xacro:include filename="$(find inail2arm_urdf)/urdf/limits.urdf.xacro" />
-    <link name="world"/>
-    <xacro:inail2_base rot="1" parent="world">
-      <origin xyz="$(arg x) $(arg y) $(arg z)" rpy="$(arg roll) $(arg pitch) $(arg yaw)"/>
+    <xacro:inail2_base rot="1" parent="$(arg parent)">
+        <origin xyz="$(arg x) $(arg y) $(arg z)" rpy="$(arg roll) $(arg pitch) $(arg yaw)"/>
     </xacro:inail2_base>
     <xacro:inail2_arm arm_num="1"  rot="1"  parent="base_link">

File: inail2arm_urdf/urdf/inail2arm_robot.urdf.xacro (robot description, xacro)
@@ -7,4 +7,10 @@
     <xacro:arg name="pitch" default="0"/>
     <xacro:arg name="yaw" default="0"/>
+    <link name="world"/>
+    <joint name="reference" type="fixed">
+      <parent link="world"/>
+      <child link="base_link"/>
+      <origin xyz="$(arg x) $(arg y) $(arg z)" rpy="$(arg roll) $(arg pitch) $(arg yaw)"/>
+    </joint>
     <!-- **** main robot model **** -->
     <xacro:include filename="$(find inail2arm_urdf)/urdf/inail2arm.urdf.xacro" />

File: inail2arm_urdf/urdf/inail2base.urdf.xacro (robot description, xacro)
@@ -27,9 +27,11 @@
         </link>
         <!-- base -->
-        <joint name="base_joint" type="fixed">
-            <parent link="${parent}" />
-            <child link="base_link" />
-            <xacro:insert_block name="origin" />
-        </joint>
+        <xacro:unless value="${parent == ''}">
+            <joint name="base_joint" type="fixed">
+                <parent link="${parent}" />
+                <child link="base_link" />
+                <xacro:insert_block name="origin" />
+            </joint>
+        </xacro:unless>
     </xacro:macro>
 </robot>

Commit message: added proximity sensors in the urdf

File: inail2arm_urdf/urdf/inail2arm.urdf (robot description, URDF)
Before this commit: robot inail2arm, 11 links, 10 joints
Links:
- added link teraflex_1_sensor1_link
- added link teraflex_1_sensor2_link
- added link teraflex_1_sensor3_link
- added link teraflex_1_sensor4_link
- added link teraflex_1_sensor5_link
- added link teraflex_1_sensor6_link
Joints:
- added joint teraflex_1_sensor0_joint: type fixed, parent arm1_4, child teraflex_1_sensor1_link, origin xyz=0.05460 -0.069500 0.0599528 rpy=-3.1416 0.0 0.0
- added joint teraflex_1_sensor1_joint: type fixed, parent arm1_4, child teraflex_1_sensor2_link, origin xyz=0.00 -0.112600 0.0599528 rpy=3.1416 0.0 -1.5708
- added joint teraflex_1_sensor2_joint: type fixed, parent arm1_4, child teraflex_1_sensor3_link, origin xyz=-0.05460 -0.069500 0.0599528 rpy=3.1416 0.0 3.1416
- added joint teraflex_1_sensor3_joint: type fixed, parent arm1_4, child teraflex_1_sensor4_link, origin xyz=0.05460 -0.1100 0.22920 rpy=3.1416 0.0 0.0
- added joint teraflex_1_sensor4_joint: type fixed, parent arm1_4, child teraflex_1_sensor5_link, origin xyz=0.0 -0.133600 0.22920 rpy=3.1416 0.0 -1.5708
- added joint teraflex_1_sensor5_joint: type fixed, parent arm1_4, child teraflex_1_sensor6_link, origin xyz=-0.05460 -0.1100 0.22920 rpy=3.1416 0.0 3.1416

Commit message: screw links can be useful

File: inail2arm_urdf/urdf/inail2arm.urdf (robot description, URDF)
Before this commit: robot inail2arm, 17 links, 16 joints
Links:
- added link screw_bottom_left
- added link screw_bottom_right
- added link screw_top_left
- added link screw_top_right
- link dagana_1_top_link: geometry collision mesh filename=package://dagana_urdf/meshes/dg0001-simplified.stl scale=0.001 0.001 0.001; visual mesh filename=package://dagana_urdf/meshes/dg0001-simplified.stl scale=0.001 0.001 0.001
Joints:
- added joint screw_bottom_left_joint: type fixed, parent base_link, child screw_bottom_left, origin xyz=-0.05 0.05 0 rpy=0 0 0
- added joint screw_bottom_right_joint: type fixed, parent base_link, child screw_bottom_right, origin xyz=-0.05 -0.05 0 rpy=0 0 0
- added joint screw_top_left_joint: type fixed, parent base_link, child screw_top_left, origin xyz=0.05 0.05 0 rpy=0 0 0
- added joint screw_top_right_joint: type fixed, parent base_link, child screw_top_right, origin xyz=0.05 -0.05 0 rpy=0 0 0

File: inail2arm_urdf/urdf/inail2arm_robot.urdf (robot description, URDF)
Before this commit: robot inail2arm, 12 links, 11 joints
Links:
- added link screw_bottom_left
- added link screw_bottom_right
- added link screw_top_left
- added link screw_top_right
- added link teraflex_1_sensor1_link
- added link teraflex_1_sensor2_link
- added link teraflex_1_sensor3_link
- added link teraflex_1_sensor4_link
- added link teraflex_1_sensor5_link
- added link teraflex_1_sensor6_link
- link dagana_1_top_link: geometry collision mesh filename=package://dagana_urdf/meshes/dg0001-simplified.stl scale=0.001 0.001 0.001; visual mesh filename=package://dagana_urdf/meshes/dg0001-simplified.stl scale=0.001 0.001 0.001
Joints:
- removed joint base_joint
- added joint reference: type fixed, parent world, child base_link, origin xyz=0 0 0 rpy=0 0 0
- added joint screw_bottom_left_joint: type fixed, parent base_link, child screw_bottom_left, origin xyz=-0.05 0.05 0 rpy=0 0 0
- added joint screw_bottom_right_joint: type fixed, parent base_link, child screw_bottom_right, origin xyz=-0.05 -0.05 0 rpy=0 0 0
- added joint screw_top_left_joint: type fixed, parent base_link, child screw_top_left, origin xyz=0.05 0.05 0 rpy=0 0 0
- added joint screw_top_right_joint: type fixed, parent base_link, child screw_top_right, origin xyz=0.05 -0.05 0 rpy=0 0 0
- added joint teraflex_1_sensor0_joint: type fixed, parent arm1_4, child teraflex_1_sensor1_link, origin xyz=0.05460 -0.069500 0.0599528 rpy=-3.1416 0.0 0.0
- added joint teraflex_1_sensor1_joint: type fixed, parent arm1_4, child teraflex_1_sensor2_link, origin xyz=0.00 -0.112600 0.0599528 rpy=3.1416 0.0 -1.5708
- added joint teraflex_1_sensor2_joint: type fixed, parent arm1_4, child teraflex_1_sensor3_link, origin xyz=-0.05460 -0.069500 0.0599528 rpy=3.1416 0.0 3.1416
- added joint teraflex_1_sensor3_joint: type fixed, parent arm1_4, child teraflex_1_sensor4_link, origin xyz=0.05460 -0.1100 0.22920 rpy=3.1416 0.0 0.0
- added joint teraflex_1_sensor4_joint: type fixed, parent arm1_4, child teraflex_1_sensor5_link, origin xyz=0.0 -0.133600 0.22920 rpy=3.1416 0.0 -1.5708
- added joint teraflex_1_sensor5_joint: type fixed, parent arm1_4, child teraflex_1_sensor6_link, origin xyz=-0.05460 -0.1100 0.22920 rpy=3.1416 0.0 3.1416

File: inail2arm_urdf/urdf/inail2base.urdf.xacro (robot description, xacro)
@@ -27,4 +27,30 @@
         </link>
         <!-- base -->
+        <!-- Screws mounting points -->
+        <link name="screw_top_right"></link>
+        <link name="screw_top_left"></link>
+        <link name="screw_bottom_right"></link>
+        <link name="screw_bottom_left"></link>
+        <joint name="screw_top_right_joint" type="fixed">
+            <parent link="base_link" />
+            <child link="screw_top_right" />
+            <origin xyz="0.05 -0.05 0" rpy="0 0 0"/>
+        </joint>
+        <joint name="screw_top_left_joint" type="fixed">
+            <parent link="base_link" />
+            <child link="screw_top_left" />
+            <origin xyz="0.05 0.05 0" rpy="0 0 0"/>
+        </joint>
+        <joint name="screw_bottom_right_joint" type="fixed">
+            <parent link="base_link" />
+            <child link="screw_bottom_right" />
+            <origin xyz="-0.05 -0.05 0" rpy="0 0 0"/>
+        </joint>
+        <joint name="screw_bottom_left_joint" type="fixed">
+            <parent link="base_link" />
+            <child link="screw_bottom_left" />
+            <origin xyz="-0.05 0.05 0" rpy="0 0 0"/>
+        </joint>
+        <!-- Screws mounting point -->
         <xacro:unless value="${parent == ''}">
             <joint name="base_joint" type="fixed">

Commit message: urdf generated with new mesh

File: inail2arm_urdf/urdf/inail2arm.urdf (robot description, URDF)
Before this commit: robot inail2arm, 18 links, 17 joints
Links:
- link arm1_6: mass 0.001 -> 0.20700511; geometry collision mesh filename=package://inail2arm_urdf/meshes/mesh_wrist-roll.stl scale=0.001 0.001 0.001; visual mesh filename=package://inail2arm_urdf/meshes/mesh_wrist-roll.stl scale=0.001 0.001 0.001
Joints:
- joint j_arm1_6: axis 0 1 0 -> 0 0 1; origin xyz=0.0 -0.02 0.043 rpy=0 0.0 0.0 -> xyz=0.0 -0.033 0.043 rpy=1.570796326795 0.0 0.0
- joint j_tcp_1: origin xyz=0 0 0 rpy=0. 0. 0. -> xyz=0.0 0.0 0.03475 rpy=0.0 0.0 0.0
