Commit message: gazebo worlds launches and specific launch for HARIA with table and cubes

File: inail2arm_urdf/urdf/inail2arm.urdf.xacro (robot description, xacro)
@@ -1,4 +1,10 @@
 <?xml version="1.0"?>
 <robot xmlns:xacro="http://ros.org/wiki/xacro" name="inail2arm">
+    <xacro:arg name="x" default="0"/>
+    <xacro:arg name="y" default="0"/>
+    <xacro:arg name="z" default="0"/>
+    <xacro:arg name="roll" default="0"/>
+    <xacro:arg name="pitch" default="0"/>
+    <xacro:arg name="yaw" default="0"/>
     <xacro:include filename="$(find inail2arm_urdf)/urdf/conversions.urdf.xacro" />
     <xacro:include filename="$(find inail2arm_urdf)/urdf/materials.urdf.xacro" />
@@ -10,5 +16,5 @@
     <link name="world"/>
     <xacro:inail2_base rot="1" parent="world">
-      <origin xyz="0 0 0" rpy="0 0 0"/>
+      <origin xyz="$(arg x) $(arg y) $(arg z)" rpy="$(arg roll) $(arg pitch) $(arg yaw)"/>
     </xacro:inail2_base>
     <xacro:inail2_arm arm_num="1"  rot="1"  parent="base_link">

Commit message: ading teraflex sensors in the urdf

File: inail2arm_urdf/urdf/inail2arm.urdf.xacro (robot description, xacro)
@@ -26,3 +26,47 @@
     <xacro:inail2_arm_ee arm_num="1"  parent="arm1_6">
     </xacro:inail2_arm_ee>
+     <!-- Proximity Sensors -->
+  <link name="teraflex_1_sensor1_link"/>
+  <link name="teraflex_1_sensor2_link"/>
+  <link name="teraflex_1_sensor3_link"/>
+  <link name="teraflex_1_sensor4_link"/>
+  <link name="teraflex_1_sensor5_link"/>
+  <link name="teraflex_1_sensor6_link"/>
+    <!-- joint fake -->
+  <joint name="teraflex_1_sensor0_joint" type="fixed"> <!-- sensor 1 -->
+    <parent link="arm1_4"/>
+    <child link="teraflex_1_sensor1_link"/>
+    <origin rpy="1.5708 0.6405 3.1416" xyz="0.05460 -0.069500 0.0599528"/>
+  </joint>
+    <!-- joint fake -->
+  <joint name="teraflex_1_sensor1_joint" type="fixed"> <!-- sensor 2 -->
+    <parent link="arm1_4"/>
+    <child link="teraflex_1_sensor2_link"/>
+    <origin rpy="1.5708 1.4259 3.1416" xyz="0.00 -0.112600 0.0599528"/>
+  </joint>
+    <!-- joint fake -->
+  <joint name="teraflex_1_sensor2_joint" type="fixed"> <!-- sensor 3 -->
+    <parent link="arm1_4"/>
+    <child link="teraflex_1_sensor3_link"/>
+    <origin rpy="-1.5708 0.9303 0.0" xyz="-0.05460 -0.069500 0.0599528"/>
+  </joint>
+    <!-- joint fake -->
+  <joint name="teraflex_1_sensor3_joint" type="fixed"> <!-- sensor 4 -->
+    <parent link="arm1_4"/>
+    <child link="teraflex_1_sensor4_link"/>
+    <origin rpy="-1.5708 0.1449 0.0" xyz="0.05460 -0.1100 0.22920"/>
+  </joint>
+    <!-- joint fake -->
+  <joint name="teraflex_1_sensor4_joint" type="fixed"> <!-- sensor 5 -->
+    <parent link="arm1_4"/>
+    <child link="teraflex_1_sensor5_link"/>
+    <origin rpy="-1.5708 -0.6405 0.0" xyz="0.0 -0.133600 0.22920"/>
+  </joint>
+    <!-- joint fake -->
+  <joint name="teraflex_1_sensor5_joint" type="fixed"> <!-- sensor 6 -->
+    <parent link="arm1_4"/>
+    <child link="teraflex_1_sensor6_link"/>
+    <origin rpy="-1.5708 -1.4259 0.0" xyz="-0.05460 -0.1100 0.22920"/>
+  </joint>
+<!-- Proximity Sensors END-->
 </robot>

Commit message: added proximity sensors frames in the urdf model of INAL 2 arm

File: inail2arm_urdf/urdf/inail2arm.urdf.xacro (robot description, xacro)
@@ -37,5 +37,5 @@
     <parent link="arm1_4"/>
     <child link="teraflex_1_sensor1_link"/>
-    <origin rpy="1.5708 0.6405 3.1416" xyz="0.05460 -0.069500 0.0599528"/>
+    <origin rpy="-3.1416 0.0 0.0" xyz="0.05460 -0.069500 0.0599528"/>
   </joint>
     <!-- joint fake -->
@@ -43,5 +43,5 @@
     <parent link="arm1_4"/>
     <child link="teraflex_1_sensor2_link"/>
-    <origin rpy="1.5708 1.4259 3.1416" xyz="0.00 -0.112600 0.0599528"/>
+    <origin rpy="3.1416 0.0 -1.5708" xyz="0.00 -0.112600 0.0599528"/>
   </joint>
     <!-- joint fake -->
@@ -49,5 +49,5 @@
     <parent link="arm1_4"/>
     <child link="teraflex_1_sensor3_link"/>
-    <origin rpy="-1.5708 0.9303 0.0" xyz="-0.05460 -0.069500 0.0599528"/>
+    <origin rpy="3.1416 0.0 3.1416" xyz="-0.05460 -0.069500 0.0599528"/>
   </joint>
     <!-- joint fake -->
@@ -55,5 +55,5 @@
     <parent link="arm1_4"/>
     <child link="teraflex_1_sensor4_link"/>
-    <origin rpy="-1.5708 0.1449 0.0" xyz="0.05460 -0.1100 0.22920"/>
+    <origin rpy="3.1416 0.0 0.0" xyz="0.05460 -0.1100 0.22920"/>
   </joint>
     <!-- joint fake -->
@@ -61,5 +61,5 @@
     <parent link="arm1_4"/>
     <child link="teraflex_1_sensor5_link"/>
-    <origin rpy="-1.5708 -0.6405 0.0" xyz="0.0 -0.133600 0.22920"/>
+    <origin rpy="3.1416 0.0 -1.5708" xyz="0.0 -0.133600 0.22920"/>
   </joint>
     <!-- joint fake -->
@@ -67,5 +67,5 @@
     <parent link="arm1_4"/>
     <child link="teraflex_1_sensor6_link"/>
-    <origin rpy="-1.5708 -1.4259 0.0" xyz="-0.05460 -0.1100 0.22920"/>
+    <origin rpy="3.1416 0.0 3.1416" xyz="-0.05460 -0.1100 0.22920"/>
   </joint>
 <!-- Proximity Sensors END-->

Commit message: proximity sensor optional

File: inail2arm_urdf/urdf/inail2arm.urdf.xacro (robot description, xacro)
@@ -26,47 +26,6 @@
     <xacro:inail2_arm_ee arm_num="1"  parent="arm1_6">
     </xacro:inail2_arm_ee>
-     <!-- Proximity Sensors -->
-  <link name="teraflex_1_sensor1_link"/>
-  <link name="teraflex_1_sensor2_link"/>
-  <link name="teraflex_1_sensor3_link"/>
-  <link name="teraflex_1_sensor4_link"/>
-  <link name="teraflex_1_sensor5_link"/>
-  <link name="teraflex_1_sensor6_link"/>
-    <!-- joint fake -->
-  <joint name="teraflex_1_sensor0_joint" type="fixed"> <!-- sensor 1 -->
-    <parent link="arm1_4"/>
-    <child link="teraflex_1_sensor1_link"/>
-    <origin rpy="-3.1416 0.0 0.0" xyz="0.05460 -0.069500 0.0599528"/>
-  </joint>
-    <!-- joint fake -->
-  <joint name="teraflex_1_sensor1_joint" type="fixed"> <!-- sensor 2 -->
-    <parent link="arm1_4"/>
-    <child link="teraflex_1_sensor2_link"/>
-    <origin rpy="3.1416 0.0 -1.5708" xyz="0.00 -0.112600 0.0599528"/>
-  </joint>
-    <!-- joint fake -->
-  <joint name="teraflex_1_sensor2_joint" type="fixed"> <!-- sensor 3 -->
-    <parent link="arm1_4"/>
-    <child link="teraflex_1_sensor3_link"/>
-    <origin rpy="3.1416 0.0 3.1416" xyz="-0.05460 -0.069500 0.0599528"/>
-  </joint>
-    <!-- joint fake -->
-  <joint name="teraflex_1_sensor3_joint" type="fixed"> <!-- sensor 4 -->
-    <parent link="arm1_4"/>
-    <child link="teraflex_1_sensor4_link"/>
-    <origin rpy="3.1416 0.0 0.0" xyz="0.05460 -0.1100 0.22920"/>
-  </joint>
-    <!-- joint fake -->
-  <joint name="teraflex_1_sensor4_joint" type="fixed"> <!-- sensor 5 -->
-    <parent link="arm1_4"/>
-    <child link="teraflex_1_sensor5_link"/>
-    <origin rpy="3.1416 0.0 -1.5708" xyz="0.0 -0.133600 0.22920"/>
-  </joint>
-    <!-- joint fake -->
-  <joint name="teraflex_1_sensor5_joint" type="fixed"> <!-- sensor 6 -->
-    <parent link="arm1_4"/>
-    <child link="teraflex_1_sensor6_link"/>
-    <origin rpy="3.1416 0.0 3.1416" xyz="-0.05460 -0.1100 0.22920"/>
-  </joint>
-<!-- Proximity Sensors END-->
+    <xacro:if value="${PROXIMITY_SENSORS}">
+        <xacro:include filename="$(find inail2arm_urdf)/urdf/inail2arm_proximity_sensors.urdf.xacro" />
+    </xacro:if>
 </robot>

Commit message: fixed bug and added last link

File: inail2arm_urdf/urdf/inail2arm.urdf.xacro (robot description, xacro)
@@ -13,5 +13,6 @@
     </xacro:inail2_base>
     <xacro:inail2_arm arm_num="1"  rot="1"  parent="base_link">
-      <origin xyz="0 0 0" rpy="0 0 0"/>
+      <origin xyz="${Shoulder_1_Ox} ${Shoulder_1_Oy} ${Shoulder_1_Oz}"
+              rpy="${Shoulder_1_roll} ${Shoulder_1_pitch} ${Shoulder_1_yaw}" />
     </xacro:inail2_arm>
 </robot>

File: inail2arm_urdf/urdf/inail2arm_macro.urdf.xacro (robot description, xacro)
@@ -117,6 +117,5 @@
                <mesh
                   filename="package://inail2arm_urdf/meshes/mesh_wrist-pitch.stl"
-                  scale="0.001
-               ${rot*0.001} 0.001" />
+                  scale="0.001 ${rot*0.001} 0.001" />
             </geometry>
             <material name="blue" />
@@ -139,23 +138,21 @@
                iyy="${Wrist_2_yy}" iyz="${rot*Wrist_2_yz}" izz="${Wrist_2_zz}" />
          </inertial>
-         <!-- <visual>
-            <origin xyz="0.0 0.0 0.0" rpy="0.0 0.0 0.0" />
-            <geometry>
-               <mesh
-                  filename="package://inail2arm_urdf/meshes/mesh_wrist-pitch.stl"
-                  scale="0.001
-               ${rot*0.001} 0.001" />
-            </geometry>
-            <material name="blue" />
-         </visual>
-         <collision>
-            <origin xyz="0.0 0.0 0.0" rpy="0.0 0.0 0.0" />
-            <geometry>
-               <mesh
-                  filename="package://inail2arm_urdf/meshes/simple/mesh_wrist-pitch.stl"
-                  scale="0.001
-               ${rot*0.001} 0.001" />
-            </geometry>
-         </collision> -->
+         <visual>
+            <origin xyz="0.0 0.0 0.0" rpy="0.0 0.0 0.0" />
+            <geometry>
+               <mesh
+                  filename="package://inail2arm_urdf/meshes/mesh_wrist-roll.stl"
+                  scale="0.001 ${rot*0.001} 0.001" />
+            </geometry>
+            <material name="blue" />
+         </visual>
+         <collision>
+            <origin xyz="0.0 0.0 0.0" rpy="0.0 0.0 0.0" />
+            <geometry>
+               <mesh
+                  filename="package://inail2arm_urdf/meshes/simple/mesh_wrist-roll.stl"
+                  scale="0.001 ${rot*0.001} 0.001" />
+            </geometry>
+         </collision>
       </link>
       <link name="tcp_${arm_num}" />
@@ -168,8 +165,7 @@
          <child link="arm${arm_num}_1" />
          <axis xyz="0 0 1" />
-         <origin xyz="${Shoulder_1_Ox} ${rot*Shoulder_1_Oy} ${Shoulder_1_Oz}"
-            rpy="${rot*Shoulder_1_roll} ${Shoulder_1_pitch} ${Shoulder_1_yaw}" />
-         <limit lower="${j_arm_1_lower[arm_num-1]}" upper="${j_arm_1_upper[arm_num-1]}"
-            effort="${j_arm_1_torque[arm_num-1]}" velocity="${j_arm_1_velocity[arm_num-1]}" />
+         <xacro:insert_block name="origin" />
+         <limit lower="${j_arm_1_lower[0]}" upper="${j_arm_1_upper[0]}"
+            effort="${j_arm_1_torque[0]}" velocity="${j_arm_1_velocity[0]}" />
       </joint>
       <!-- shoulder yaw -->
@@ -181,6 +177,6 @@
             rpy="${rot*Shoulder_2_roll} ${Shoulder_2_pitch} ${Shoulder_2_yaw}" />
          <axis xyz="0 0 -1" />
-         <limit lower="${j_arm_2_lower[arm_num-1]}" upper="${j_arm_2_upper[arm_num-1]}"
-            effort="${j_arm_2_torque[arm_num-1]}" velocity="${j_arm_2_velocity[arm_num-2]}" />
+         <limit lower="${j_arm_2_lower[0]}" upper="${j_arm_2_upper[0]}"
+            effort="${j_arm_2_torque[0]}" velocity="${j_arm_2_velocity[0]}" />
       </joint>
       <!-- shoulder pitch -->
@@ -192,6 +188,6 @@
             rpy="${rot*Elbow_1_roll} ${Elbow_1_pitch} ${Elbow_1_yaw}" />
          <axis xyz="0 0 1" />
-         <limit lower="${j_arm_3_lower[arm_num-1]}" upper="${j_arm_3_upper[arm_num-1]}"
-            effort="${j_arm_3_torque[arm_num-1]}" velocity="${j_arm_3_velocity[arm_num-1]}" />
+         <limit lower="${j_arm_3_lower[0]}" upper="${j_arm_3_upper[0]}"
+            effort="${j_arm_3_torque[0]}" velocity="${j_arm_3_velocity[0]}" />
       </joint>
       <!-- elbow yaw -->
@@ -200,9 +196,9 @@
          <parent link="arm${arm_num}_3" />
          <child link="arm${arm_num}_4" />
-         <origin xyz="${Forearm_1_Ox} ${Forearm_1_Oy} ${Forearm_1_Oz}"
+         <origin xyz="${Forearm_1_Ox} ${rot*Forearm_1_Oy} ${Forearm_1_Oz}"
             rpy="${rot*Forearm_1_roll} ${Forearm_1_pitch} ${Forearm_1_yaw}" />
          <axis xyz="0 0 1" />
-         <limit lower="${j_arm_4_lower[arm_num-1]}" upper="${j_arm_4_upper[arm_num-1]}"
-            effort="${j_arm_4_torque[arm_num-1]}" velocity="${j_arm_4_velocity[arm_num-1]}" />
+         <limit lower="${j_arm_4_lower[0]}" upper="${j_arm_4_upper[0]}"
+            effort="${j_arm_4_torque[0]}" velocity="${j_arm_4_velocity[0]}" />
       </joint>
       <!-- forearm yaw -->
@@ -214,9 +210,9 @@
             rpy="${rot*Wrist_1_roll} ${Wrist_1_pitch} ${Wrist_1_yaw}" />
          <axis xyz="0 0 1" />
-         <limit lower="${j_arm_5_lower[arm_num-1]}" upper="${j_arm_5_upper[arm_num-1]}"
-            effort="${j_arm_5_torque[arm_num-1]}" velocity="${j_arm_5_velocity[arm_num-1]}" />
+         <limit lower="${j_arm_5_lower[0]}" upper="${j_arm_5_upper[0]}"
+            effort="${j_arm_5_torque[0]}" velocity="${j_arm_5_velocity[0]}" />
       </joint>
       <!-- wrist pitch-->
-      <!-- wrist2 pitch-->
+      <!-- wrist2 roll-->
       <joint name="j_arm${arm_num}_6" type="revolute">
          <parent link="arm${arm_num}_5" />
@@ -224,14 +220,15 @@
          <origin xyz="${Wrist_2_Ox} ${rot*Wrist_2_Oy} ${Wrist_2_Oz}"
             rpy="${rot*Wrist_2_roll} ${Wrist_2_pitch} ${Wrist_2_yaw}" />
-         <axis xyz="0 1 0" />
-         <limit lower="${j_arm_6_lower[arm_num-1]}" upper="${j_arm_6_upper[arm_num-1]}"
-            effort="${j_arm_6_torque[arm_num-1]}" velocity="${j_arm_6_velocity[arm_num-1]}" />
-      </joint>
-      <!-- /wrist2 pitch-->
+         <axis xyz="0 0 1" />
+         <limit lower="${j_arm_6_lower[0]}" upper="${j_arm_6_upper[0]}"
+            effort="${j_arm_6_torque[0]}" velocity="${j_arm_6_velocity[0]}" />
+      </joint>
+      <!-- /wrist2 roll-->
       <!-- virtual tip pitch-->
       <joint name="j_tcp_${arm_num}" type="fixed">
          <parent link="arm${arm_num}_6" />
          <child link="tcp_${arm_num}" />
-         <origin xyz="0.0 0.0 0" />
+         <origin xyz="${No_end_ft_Ox} ${rot*No_end_ft_Oy} ${No_end_ft_Oz}"
+            rpy="${rot*No_end_ft_roll} ${No_end_ft_pitch} ${No_end_ft_yaw}" />
       </joint>
       <!-- virtual tip pitch-->

File: inail2arm_urdf/urdf/kinematics_properties.urdf.xacro (robot description, xacro)
@@ -38,7 +38,7 @@
 <!-- Origin -->
 <xacro:property name="Wrist_2_Ox" value=" 0.0 "/>
-<xacro:property name="Wrist_2_Oy" value=" -0.02 "/>
+<xacro:property name="Wrist_2_Oy" value=" -0.033 "/>
 <xacro:property name="Wrist_2_Oz" value=" 0.043 "/>
-<xacro:property name="Wrist_2_roll" value=" 0"/>
+<xacro:property name="Wrist_2_roll" value=" ${PI/2} "/>
 <xacro:property name="Wrist_2_pitch" value=" 0.0 "/>
 <xacro:property name="Wrist_2_yaw" value=" 0.0 "/>
@@ -47,5 +47,5 @@
 <xacro:property name="No_end_ft_Ox" value=" 0.0 "/>
 <xacro:property name="No_end_ft_Oy" value=" 0.0 "/>
-<xacro:property name="No_end_ft_Oz" value=" 0.0 "/>
+<xacro:property name="No_end_ft_Oz" value=" 0.03475 "/>
 <xacro:property name="No_end_ft_roll" value=" 0.0 "/>
 <xacro:property name="No_end_ft_pitch" value=" 0.0 "/>

File: inail2arm_urdf/urdf/limits.urdf.xacro (robot description, xacro)
@@ -14,16 +14,16 @@
 <xacro:property name="j_arm_5_upper" value="${[2.2]}"/>
 <xacro:property name="j_arm_6_upper" value="${[2.85]}"/>
-<xacro:property name="j_arm_1_velocity" value="${[3.86, 3.86 ]}"/>
-<xacro:property name="j_arm_2_velocity" value="${[3.86, 3.86 ]}"/>
-<xacro:property name="j_arm_3_velocity" value="${[6.06, 6.06 ]}"/>
-<xacro:property name="j_arm_4_velocity" value="${[6.06, 6.06 ]}"/>
-<xacro:property name="j_arm_5_velocity" value="${[11.72, 11.72 ]}"/>
-<xacro:property name="j_arm_6_velocity" value="${[11.72, 11.72 ]}"/>
-<xacro:property name="j_arm_1_torque" value="${[147.00, 147.00 ]}"/>
-<xacro:property name="j_arm_2_torque" value="${[147.00, 147.00 ]}"/>
-<xacro:property name="j_arm_3_torque" value="${[147.00, 147.00 ]}"/>
-<xacro:property name="j_arm_4_torque" value="${[147.00, 147.00 ]}"/>
-<xacro:property name="j_arm_5_torque" value="${[55.00, 55.00 ]}"/>
-<xacro:property name="j_arm_6_torque" value="${[55.00, 55.00 ]}"/>
+<xacro:property name="j_arm_1_velocity" value="${[3.86]}"/>
+<xacro:property name="j_arm_2_velocity" value="${[3.86]}"/>
+<xacro:property name="j_arm_3_velocity" value="${[6.06]}"/>
+<xacro:property name="j_arm_4_velocity" value="${[6.06]}"/>
+<xacro:property name="j_arm_5_velocity" value="${[11.72]}"/>
+<xacro:property name="j_arm_6_velocity" value="${[11.72]}"/>
+<xacro:property name="j_arm_1_torque" value="${[147.00]}"/>
+<xacro:property name="j_arm_2_torque" value="${[147.00]}"/>
+<xacro:property name="j_arm_3_torque" value="${[147.00]}"/>
+<xacro:property name="j_arm_4_torque" value="${[147.00]}"/>
+<xacro:property name="j_arm_5_torque" value="${[55.00]}"/>
+<xacro:property name="j_arm_6_torque" value="${[55.00]}"/>
 <xacro:property name="motor_A_velocity" value="8.8"/>
 <xacro:property name="motor_B_velocity" value="8.1"/>
