Commit message: fix: first joint's origin is set by macro argument!

File: inail2arm_urdf/urdf/inail2arm_macro.urdf.xacro (robot description, xacro)
@@ -165,8 +165,7 @@
          <child link="arm${arm_num}_1" />
          <axis xyz="0 0 1" />
-         <origin xyz="${Shoulder_1_Ox} ${rot*Shoulder_1_Oy} ${Shoulder_1_Oz}"
-            rpy="${rot*Shoulder_1_roll} ${Shoulder_1_pitch} ${Shoulder_1_yaw}" />
-         <limit lower="${j_arm_1_lower[arm_num-1]}" upper="${j_arm_1_upper[arm_num-1]}"
-            effort="${j_arm_1_torque[arm_num-1]}" velocity="${j_arm_1_velocity[arm_num-1]}" />
+         <xacro:insert_block name="origin"/>
+         <limit lower="${j_arm_1_lower[0]}" upper="${j_arm_1_upper[0]}"
+            effort="${j_arm_1_torque[0]}" velocity="${j_arm_1_velocity[0]}" />
       </joint>
       <!-- shoulder yaw -->
@@ -178,6 +177,6 @@
             rpy="${rot*Shoulder_2_roll} ${Shoulder_2_pitch} ${Shoulder_2_yaw}" />
          <axis xyz="0 0 -1" />
-         <limit lower="${j_arm_2_lower[arm_num-1]}" upper="${j_arm_2_upper[arm_num-1]}"
-            effort="${j_arm_2_torque[arm_num-1]}" velocity="${j_arm_2_velocity[arm_num-2]}" />
+         <limit lower="${j_arm_2_lower[0]}" upper="${j_arm_2_upper[0]}"
+            effort="${j_arm_2_torque[0]}" velocity="${j_arm_2_velocity[arm_num-2]}" />
       </joint>
       <!-- shoulder pitch -->
@@ -189,6 +188,6 @@
             rpy="${rot*Elbow_1_roll} ${Elbow_1_pitch} ${Elbow_1_yaw}" />
          <axis xyz="0 0 1" />
-         <limit lower="${j_arm_3_lower[arm_num-1]}" upper="${j_arm_3_upper[arm_num-1]}"
-            effort="${j_arm_3_torque[arm_num-1]}" velocity="${j_arm_3_velocity[arm_num-1]}" />
+         <limit lower="${j_arm_3_lower[0]}" upper="${j_arm_3_upper[0]}"
+            effort="${j_arm_3_torque[0]}" velocity="${j_arm_3_velocity[0]}" />
       </joint>
       <!-- elbow yaw -->
@@ -200,6 +199,6 @@
             rpy="${rot*Forearm_1_roll} ${Forearm_1_pitch} ${Forearm_1_yaw}" />
          <axis xyz="0 0 1" />
-         <limit lower="${j_arm_4_lower[arm_num-1]}" upper="${j_arm_4_upper[arm_num-1]}"
-            effort="${j_arm_4_torque[arm_num-1]}" velocity="${j_arm_4_velocity[arm_num-1]}" />
+         <limit lower="${j_arm_4_lower[0]}" upper="${j_arm_4_upper[0]}"
+            effort="${j_arm_4_torque[0]}" velocity="${j_arm_4_velocity[0]}" />
       </joint>
       <!-- forearm yaw -->
@@ -211,6 +210,6 @@
             rpy="${rot*Wrist_1_roll} ${Wrist_1_pitch} ${Wrist_1_yaw}" />
          <axis xyz="0 0 1" />
-         <limit lower="${j_arm_5_lower[arm_num-1]}" upper="${j_arm_5_upper[arm_num-1]}"
-            effort="${j_arm_5_torque[arm_num-1]}" velocity="${j_arm_5_velocity[arm_num-1]}" />
+         <limit lower="${j_arm_5_lower[0]}" upper="${j_arm_5_upper[0]}"
+            effort="${j_arm_5_torque[0]}" velocity="${j_arm_5_velocity[0]}" />
       </joint>
       <!-- wrist pitch-->
@@ -222,6 +221,6 @@
             rpy="${rot*Wrist_2_roll} ${Wrist_2_pitch} ${Wrist_2_yaw}" />
          <axis xyz="0 0 1" />
-         <limit lower="${j_arm_6_lower[arm_num-1]}" upper="${j_arm_6_upper[arm_num-1]}"
-            effort="${j_arm_6_torque[arm_num-1]}" velocity="${j_arm_6_velocity[arm_num-1]}" />
+         <limit lower="${j_arm_6_lower[0]}" upper="${j_arm_6_upper[0]}"
+            effort="${j_arm_6_torque[0]}" velocity="${j_arm_6_velocity[0]}" />
       </joint>
       <!-- /wrist2 pitch-->

Commit message: limited elbow rotation to avoid elbow flip

File: inail2arm_urdf/urdf/inail2arm_macro.urdf.xacro (robot description, xacro)
@@ -188,7 +188,16 @@
             rpy="${rot*Elbow_1_roll} ${Elbow_1_pitch} ${Elbow_1_yaw}" />
          <axis xyz="0 0 1" />
-         <limit lower="${j_arm_3_lower[0]}" upper="${j_arm_3_upper[0]}"
-            effort="${j_arm_3_torque[0]}" velocity="${j_arm_3_velocity[0]}" />
-      </joint>
+         <!-- original elbow limits
+            <limit lower="${j_arm_3_lower[0]}" upper="${j_arm_3_upper[0]}"
+         effort="${j_arm_3_torque[0]}" velocity="${j_arm_3_velocity[0]}" />
+         -->
+         <!-- Virtual limits for elbow joints, so elbow doesnt flip in undesired orientation -->
+        <xacro:if value="${parent == 'mount_frame_1'}">
+            <limit lower="${j_arm_3_lower[0]}" upper="0" effort="${j_arm_3_torque[0]}" velocity="${j_arm_3_velocity[0]}" />
+        </xacro:if>
+        <xacro:if value="${parent == 'mount_frame_2'}">
+            <limit lower="0" upper="${j_arm_3_upper[0]}" effort="${j_arm_3_torque[0]}" velocity="${j_arm_3_velocity[0]}" />
+       </xacro:if>
+    </joint>
       <!-- elbow yaw -->
       <!-- forearm yaw -->
