Commit message: corrected dagana name

File: inail2arm_urdf/urdf/gazebo/xbot.gazebo.xacro (robot description, xacro)
@@ -5,6 +5,6 @@
     <xacro:if value="${DAGANA_STANDALONE_PLUGIN}">
         <plugin filename="libdagana_gazebo_DaganaPlugin.so" name="dagana_plugin">
-            <gripperName>dagana_2</gripperName>
-            <jointName>dagana_2_claw_joint</jointName>
+            <gripperName>dagana_1</gripperName>
+            <jointName>dagana_1_claw_joint</jointName>
             <rate>100</rate>
             <p>1</p>
@@ -20,5 +20,5 @@
         <xacro:if value="${DAGANA_STANDALONE_PLUGIN}">
         <ignore_joints>
-            <joint name="dagana_2_claw_joint" />
+            <joint name="dagana_1_claw_joint" />
         </ignore_joints>
         </xacro:if>
@@ -29,4 +29,5 @@
             <gain name="medium_mot" p="4000" d="40"/>
             <gain name="big_mot"    p="8000" d="50"/>
+            <gain name="dagana_mot"  p="10" d="0.5"/>
             <pid name="j_arm1_1" profile="small_mot"/>
             <pid name="j_arm1_2" profile="small_mot"/>
@@ -35,4 +36,5 @@
             <pid name="j_arm1_5" profile="small_mot"/>
             <pid name="j_arm1_6" profile="small_mot"/>
+            <pid name="dagana_1_claw_joint" profile="dagana_mot"/>
         </pid>
     </plugin>
