Commit message: gazebo and cartesio files

File: inail2arm_urdf/urdf/gazebo/inail2arm.gazebo.xacro (robot description, xacro)
@@ -25,3 +25,27 @@
     <provideFeedback>true</provideFeedback>
 </gazebo>
+<gazebo reference="j_arm2_1">
+    <implicitSpringDamper>1</implicitSpringDamper>
+    <provideFeedback>true</provideFeedback>
+</gazebo>
+<gazebo reference="j_arm2_2">
+    <implicitSpringDamper>1</implicitSpringDamper>
+    <provideFeedback>true</provideFeedback>
+</gazebo>
+<gazebo reference="j_arm2_3">
+    <implicitSpringDamper>1</implicitSpringDamper>
+    <provideFeedback>true</provideFeedback>
+</gazebo>
+<gazebo reference="j_arm2_4">
+    <implicitSpringDamper>1</implicitSpringDamper>
+    <provideFeedback>true</provideFeedback>
+</gazebo>
+<gazebo reference="j_arm2_5">
+    <implicitSpringDamper>1</implicitSpringDamper>
+    <provideFeedback>true</provideFeedback>
+</gazebo>
+<gazebo reference="j_arm2_6">
+    <implicitSpringDamper>1</implicitSpringDamper>
+    <provideFeedback>true</provideFeedback>
+</gazebo>
 </robot>

File: inail2arm_urdf/urdf/gazebo/materials.gazebo.xacro (robot description, xacro)
@@ -1,35 +1,53 @@
 <?xml version="1.0"?>
 <robot xmlns:xacro="http://ros.org/wiki/xacro">
-<!-- **** gazebo materials **** -->
-<gazebo reference="arm1_1">
-  <material>Gazebo/Blue</material>
-</gazebo>
-<gazebo reference="arm1_2">
-  <material>Gazebo/DarkGrey</material>
-</gazebo>
-<gazebo reference="arm1_3">
-  <material>Gazebo/Blue</material>
-</gazebo>
-<gazebo reference="arm1_4">
-  <material>Gazebo/Blue</material>
-</gazebo>
-<gazebo reference="arm1_5">
-  <material>Gazebo/Blue</material>
-</gazebo>
-<gazebo reference="arm1_6">
-  <material>Gazebo/Blue</material>
-</gazebo>
-<xacro:if value="${END_EFFECTOR == 'ball'}">
-	<gazebo reference="ball1">
-		<material>Gazebo/BlackTransparent</material>
+	<!-- **** gazebo materials **** -->
+	<gazebo reference="arm1_1">
+		<material>Gazebo/Blue</material>
 	</gazebo>
-</xacro:if>
-<xacro:if value="${END_EFFECTOR == 'dagana' or END_EFFECTOR == 'dagana_fixed'}">
-	<gazebo reference="dagana_1_top_link">
-		<material>Gazebo/BlackTransparent</material>
+	<gazebo reference="arm1_2">
+		<material>Gazebo/DarkGrey</material>
 	</gazebo>
-	<gazebo reference="dagana_1_bottom_link">
-		<material>Gazebo/BlackTransparent</material>
+	<gazebo reference="arm1_3">
+		<material>Gazebo/Blue</material>
 	</gazebo>
-</xacro:if>
+	<gazebo reference="arm1_4">
+		<material>Gazebo/Blue</material>
+	</gazebo>
+	<gazebo reference="arm1_5">
+		<material>Gazebo/Blue</material>
+	</gazebo>
+	<gazebo reference="arm1_6">
+		<material>Gazebo/Blue</material>
+	</gazebo>
+	<gazebo reference="arm2_1">
+		<material>Gazebo/Blue</material>
+	</gazebo>
+	<gazebo reference="arm2_2">
+		<material>Gazebo/DarkGrey</material>
+	</gazebo>
+	<gazebo reference="arm2_3">
+		<material>Gazebo/Blue</material>
+	</gazebo>
+	<gazebo reference="arm2_4">
+		<material>Gazebo/Blue</material>
+	</gazebo>
+	<gazebo reference="arm2_5">
+		<material>Gazebo/Blue</material>
+	</gazebo>
+	<gazebo reference="arm2_6">
+		<material>Gazebo/Blue</material>
+	</gazebo>
+	<xacro:if value="${END_EFFECTOR == 'ball'}">
+		<gazebo reference="ball1">
+			<material>Gazebo/BlackTransparent</material>
+		</gazebo>
+	</xacro:if>
+	<xacro:if value="${END_EFFECTOR == 'dagana' or END_EFFECTOR == 'dagana_fixed'}">
+		<gazebo reference="dagana_1_top_link">
+			<material>Gazebo/BlackTransparent</material>
+		</gazebo>
+		<gazebo reference="dagana_1_bottom_link">
+			<material>Gazebo/BlackTransparent</material>
+		</gazebo>
+	</xacro:if>
 </robot>

File: inail2arm_urdf/urdf/gazebo/xbot.gazebo.xacro (robot description, xacro)
@@ -37,4 +37,10 @@
             <pid name="j_arm1_6" profile="small_mot"/>
             <pid name="dagana_1_claw_joint" profile="dagana_mot"/>
+            <pid name="j_arm2_1" profile="small_mot"/>
+            <pid name="j_arm2_2" profile="small_mot"/>
+            <pid name="j_arm2_3" profile="small_mot"/>
+            <pid name="j_arm2_4" profile="small_mot"/>
+            <pid name="j_arm2_5" profile="small_mot"/>
+            <pid name="j_arm2_6" profile="small_mot"/>
         </pid>
     </plugin>
