Commit message: updates

File: inail2arm_srdf/srdf/inail2arm.srdf.xacro (robot description, xacro)
@@ -2,5 +2,5 @@
 <robot name="inail2arm">
     <group name="arm">
-        <chain base_link="base_link" tip_link="arm1_5" />
+        <chain base_link="base_link" tip_link="arm1_6" />
     </group>
     <group name="chains">
@@ -13,4 +13,5 @@
         <joint name="j_arm1_4" value="0.0" />
         <joint name="j_arm1_5" value="0.0" />
+        <joint name="j_arm1_6" value="0.0" />
     </group_state>
     <!-- <disable_collisions link1="arm1_1" link2="arm1_2" reason="Never" /> -->

File: inail2arm_urdf/urdf/inail2arm.urdf.xacro (robot description, xacro)
@@ -132,4 +132,31 @@
          </collision>
       </link>
+      <link name="arm${arm_num}_6">
+         <inertial>
+            <origin xyz="${Wrist_2_x} ${rot*Wrist_2_y} ${Wrist_2_z}" />
+            <mass value="${Wrist_2_mass}" />
+            <inertia ixx="${Wrist_2_xx}" ixy="${rot*Wrist_2_xy}" ixz="${Wrist_2_xz}"
+               iyy="${Wrist_2_yy}" iyz="${rot*Wrist_2_yz}" izz="${Wrist_2_zz}" />
+         </inertial>
+         <!-- <visual>
+            <origin xyz="0.0 0.0 0.0" rpy="0.0 0.0 0.0" />
+            <geometry>
+               <mesh
+                  filename="package://inail2arm_urdf/meshes/mesh_wrist-pitch.stl"
+                  scale="0.001
+               ${rot*0.001} 0.001" />
+            </geometry>
+            <material name="blue" />
+         </visual>
+         <collision>
+            <origin xyz="0.0 0.0 0.0" rpy="0.0 0.0 0.0" />
+            <geometry>
+               <mesh
+                  filename="package://inail2arm_urdf/meshes/simple/mesh_wrist-pitch.stl"
+                  scale="0.001
+               ${rot*0.001} 0.001" />
+            </geometry>
+         </collision> -->
+      </link>
       <!--wrist-pitch -->
       <!-- /LINKS -->
@@ -152,5 +179,5 @@
          <origin xyz="${Shoulder_2_Ox} ${rot*Shoulder_2_Oy} ${Shoulder_2_Oz}"
             rpy="${rot*Shoulder_2_roll} ${Shoulder_2_pitch} ${Shoulder_2_yaw}" />
-         <axis xyz="0 0 1" />
+         <axis xyz="0 0 -1" />
          <limit lower="${j_arm_2_lower[arm_num-1]}" upper="${j_arm_2_upper[arm_num-1]}"
             effort="${j_arm_2_torque[arm_num-1]}" velocity="${j_arm_2_velocity[arm_num-2]}" />
@@ -191,13 +218,13 @@
       <!-- wrist pitch-->
       <!-- wrist2 pitch-->
-      <!-- <joint name="j_arm${arm_num}_6" type="revolute">
+      <joint name="j_arm${arm_num}_6" type="revolute">
          <parent link="arm${arm_num}_5" />
          <child link="arm${arm_num}_6" />
-         <origin xyz="${Wrist_1_Ox} ${rot*Wrist_1_Oy} ${Wrist_1_Oz}"
-               rpy="${rot*Wrist_1_roll} ${Wrist_1_pitch} ${Wrist_1_yaw}" />
+         <origin xyz="${Wrist_2_Ox} ${rot*Wrist_2_Oy} ${Wrist_2_Oz}"
+               rpy="${rot*Wrist_2_roll} ${Wrist_2_pitch} ${Wrist_2_yaw}" />
          <axis xyz="0 0 1" />
          <limit lower="${j_arm_6_lower[arm_num-1]}" upper="${j_arm_6_upper[arm_num-1]}"
             effort="${j_arm_6_torque[arm_num-1]}" velocity="${j_arm_6_velocity[arm_num-1]}" />
-      </joint> -->
+      </joint>
       <!-- /wrist2 pitch-->
    </xacro:macro>

File: inail2arm_urdf/urdf/inertial_properties.urdf.xacro (robot description, xacro)
@@ -86,15 +86,15 @@
 <xacro:property name="Wrist_1_mass" value=" 1.0418416 "/>
 <!-- Center of Mass -->
-<xacro:property name="Wrist_2_x" value=" "/>
-<xacro:property name="Wrist_2_y" value=" "/>
-<xacro:property name="Wrist_2_z" value=" "/>
+<xacro:property name="Wrist_2_x" value="0 "/>
+<xacro:property name="Wrist_2_y" value="0 "/>
+<xacro:property name="Wrist_2_z" value="0 "/>
 <!-- Inertia -->
-<xacro:property name="Wrist_2_xx" value=" "/>
-<xacro:property name="Wrist_2_yy" value=" "/>
-<xacro:property name="Wrist_2_zz" value=" "/>
-<xacro:property name="Wrist_2_xy" value=" "/>
-<xacro:property name="Wrist_2_xz" value=" "/>
-<xacro:property name="Wrist_2_yz" value=" "/>
+<xacro:property name="Wrist_2_xx" value="0.0001 "/>
+<xacro:property name="Wrist_2_yy" value="0.0001 "/>
+<xacro:property name="Wrist_2_zz" value="0.0001 "/>
+<xacro:property name="Wrist_2_xy" value="0 "/>
+<xacro:property name="Wrist_2_xz" value="0"/>
+<xacro:property name="Wrist_2_yz" value="0"/>
 <!-- Mass -->
-<xacro:property name="Wrist_2_mass" value=" "/>
+<xacro:property name="Wrist_2_mass" value="0.001 "/>
 </robot>

File: inail2arm_urdf/urdf/kinematics_properties.urdf.xacro (robot description, xacro)
@@ -36,4 +36,11 @@
 <xacro:property name="Wrist_1_pitch" value=" 0.0 "/>
 <xacro:property name="Wrist_1_yaw" value=" 0.0 "/>
+<!-- Origin -->
+<xacro:property name="Wrist_2_Ox" value=" 0.0 "/>
+<xacro:property name="Wrist_2_Oy" value=" -0.0 "/>
+<xacro:property name="Wrist_2_Oz" value=" 0.0 "/>
+<xacro:property name="Wrist_2_roll" value=" 0"/>
+<xacro:property name="Wrist_2_pitch" value=" 0.0 "/>
+<xacro:property name="Wrist_2_yaw" value=" 0.0 "/>
 <!-- END-EFFECTORS-->
 <!-- Origin -->

Commit message: added cartesio simulation for inail2arm

File: inail2arm_srdf/srdf/inail2arm.srdf.xacro (robot description, xacro)
@@ -9,8 +9,8 @@
     <group_state name="home" group="chains">
         <joint name="j_arm1_1" value="0.0" />
-        <joint name="j_arm1_2" value="0.0" />
-        <joint name="j_arm1_3" value="0.0" />
+        <joint name="j_arm1_2" value="0.45" />
+        <joint name="j_arm1_3" value="-1.6" />
         <joint name="j_arm1_4" value="0.0" />
-        <joint name="j_arm1_5" value="0.0" />
+        <joint name="j_arm1_5" value="1.1" />
         <joint name="j_arm1_6" value="0.0" />
     </group_state>

File: inail2arm_urdf/urdf/inail2arm.urdf.xacro (robot description, xacro)
@@ -1,232 +1,17 @@
 <?xml version="1.0"?>
-<robot xmlns:xacro="http://ros.org/wiki/xacro">
-   <!-- macro arms -->
-   <xacro:macro name="inail2_arm" params="arm_num rot parent *origin">
-      <!-- LINKS -->
-      <!-- shoulder yaw-->
-      <link name="arm${arm_num}_1">
-         <inertial>
-            <origin xyz="${Shoulder_1_x} ${rot*Shoulder_1_y} ${Shoulder_1_z}" />
-            <mass value="${Shoulder_1_mass}" />
-            <inertia ixx="${Shoulder_1_xx}" ixy="${rot*Shoulder_1_xy}" ixz="${Shoulder_1_xz}"
-               iyy="${Shoulder_1_yy}" iyz="${rot*Shoulder_1_yz}" izz="${Shoulder_1_zz}" />
-         </inertial>
-         <visual>
-            <origin xyz="0.0 0.0 0.0" rpy="0.0 0.0 0.0" />
-            <geometry>
-               <mesh filename="package://inail2arm_urdf/meshes/mesh_shoulder-yaw.stl"
-                  scale="0.001 ${rot*0.001} 0.001" />
-            </geometry>
-            <material name="blue" />
-         </visual>
-         <collision>
-            <origin xyz="0.0 0.0 0.0" rpy="0.0 0.0 0.0" />
-            <geometry>
-               <mesh filename="package://inail2arm_urdf/meshes/simple/mesh_shoulder-yaw.stl"
-                  scale="0.001 ${rot*0.001} 0.001" />
-            </geometry>
-         </collision>
-      </link>
-      <!-- shoulder yaw-->
-      <!-- shoulder pitch-->
-      <link name="arm${arm_num}_2">
-         <inertial>
-            <origin xyz="${Shoulder_2_x} ${rot*Shoulder_2_y} ${Shoulder_2_z}" />
-            <mass value="${Shoulder_2_mass}" />
-            <inertia ixx="${Shoulder_2_xx}" ixy="${rot*Shoulder_2_xy}" ixz="${Shoulder_2_xz}"
-               iyy="${Shoulder_2_yy}" iyz="${rot*Shoulder_2_yz}" izz="${Shoulder_2_zz}" />
-         </inertial>
-         <visual>
-            <origin xyz="0.0 0.0 0.0" rpy="0.0 0.0 0.0" />
-            <geometry>
-               <mesh filename="package://inail2arm_urdf/meshes/mesh_shoulder-pitch.stl"
-                  scale="0.001 ${rot*0.001} 0.001" />
-            </geometry>
-            <material name="blue" />
-         </visual>
-         <collision>
-            <origin xyz="0.0 0.0 0.0" rpy="0.0 0.0 0.0" />
-            <geometry>
-               <mesh filename="package://inail2arm_urdf/meshes/simple/mesh_shoulder-pitch.stl"
-                  scale="0.001 ${rot*0.001} 0.001" />
-            </geometry>
-         </collision>
-      </link>
-      <!-- shoulder pitch-->
-      <!-- elbow-yaw-->
-      <link name="arm${arm_num}_3">
-         <inertial>
-            <origin xyz="${Elbow_1_x} ${rot*Elbow_1_y} ${Elbow_1_z}" />
-            <mass value="${Elbow_1_mass}" />
-            <inertia ixx="${Elbow_1_xx}" ixy="${rot*Elbow_1_xy}" ixz="${Elbow_1_xz}"
-               iyy="${Elbow_1_yy}" iyz="${rot*Elbow_1_yz}" izz="${Elbow_1_zz}" />
-         </inertial>
-         <visual>
-            <origin xyz="0.0 0.0 0.0" rpy="0.0 0.0 0.0" />
-            <geometry>
-               <mesh filename="package://inail2arm_urdf/meshes/mesh_elbow.stl"
-                  scale="0.001 ${rot*0.001} 0.001" />
-            </geometry>
-            <material name="blue" />
-         </visual>
-         <collision>
-            <origin xyz="0.0 0.0 0.0" rpy="0.0 0.0 0.0" />
-            <geometry>
-               <mesh filename="package://inail2arm_urdf/meshes/simple/mesh_elbow.stl"
-                  scale="0.001 ${rot*0.001} 0.001" />
-            </geometry>
-         </collision>
-      </link>
-      <!-- elbow-yaw-->
-      <!-- forearm-yaw -->
-      <link name="arm${arm_num}_4">
-         <inertial>
-            <origin xyz="${Forearm_1_x} ${rot*Forearm_1_y} ${Forearm_1_z}" />
-            <mass value="${Forearm_1_mass}" />
-            <inertia ixx="${Forearm_1_xx}" ixy="${rot*Forearm_1_xy}" ixz="${Forearm_1_xz}"
-               iyy="${Forearm_1_yy}" iyz="${rot*Forearm_1_yz}" izz="${Forearm_1_zz}" />
-         </inertial>
-         <visual>
-            <origin xyz="0.0 0.0 0.0" rpy="0.0 0.0 0.0" />
-            <geometry>
-               <mesh filename="package://inail2arm_urdf/meshes/mesh_forearm-yaw.stl"
-                  scale="0.001 ${rot*0.001} 0.001" />
-            </geometry>
-            <material name="blue" />
-         </visual>
-         <collision>
-            <origin xyz="0.0 0.0 0.0" rpy="0.0 0.0 0.0" />
-            <geometry>
-               <mesh filename="package://inail2arm_urdf/meshes/simple/mesh_forearm-yaw.stl"
-                  scale="0.001 ${rot*0.001} 0.001" />
-            </geometry>
-         </collision>
-      </link>
-      <!-- forearm-yaw -->
-      <!--wrist-pitch -->
-      <link name="arm${arm_num}_5">
-         <inertial>
-            <origin xyz="${Wrist_1_x} ${rot*Wrist_1_y} ${Wrist_1_z}" />
-            <mass value="${Wrist_1_mass}" />
-            <inertia ixx="${Wrist_1_xx}" ixy="${rot*Wrist_1_xy}" ixz="${Wrist_1_xz}"
-               iyy="${Wrist_1_yy}" iyz="${rot*Wrist_1_yz}" izz="${Wrist_1_zz}" />
-         </inertial>
-         <visual>
-            <origin xyz="0.0 0.0 0.0" rpy="0.0 0.0 0.0" />
-            <geometry>
-               <mesh
-                  filename="package://inail2arm_urdf/meshes/mesh_wrist-pitch.stl"
-                  scale="0.001
-               ${rot*0.001} 0.001" />
-            </geometry>
-            <material name="blue" />
-         </visual>
-         <collision>
-            <origin xyz="0.0 0.0 0.0" rpy="0.0 0.0 0.0" />
-            <geometry>
-               <mesh
-                  filename="package://inail2arm_urdf/meshes/simple/mesh_wrist-pitch.stl"
-                  scale="0.001
-               ${rot*0.001} 0.001" />
-            </geometry>
-         </collision>
-      </link>
-      <link name="arm${arm_num}_6">
-         <inertial>
-            <origin xyz="${Wrist_2_x} ${rot*Wrist_2_y} ${Wrist_2_z}" />
-            <mass value="${Wrist_2_mass}" />
-            <inertia ixx="${Wrist_2_xx}" ixy="${rot*Wrist_2_xy}" ixz="${Wrist_2_xz}"
-               iyy="${Wrist_2_yy}" iyz="${rot*Wrist_2_yz}" izz="${Wrist_2_zz}" />
-         </inertial>
-         <!-- <visual>
-            <origin xyz="0.0 0.0 0.0" rpy="0.0 0.0 0.0" />
-            <geometry>
-               <mesh
-                  filename="package://inail2arm_urdf/meshes/mesh_wrist-pitch.stl"
-                  scale="0.001
-               ${rot*0.001} 0.001" />
-            </geometry>
-            <material name="blue" />
-         </visual>
-         <collision>
-            <origin xyz="0.0 0.0 0.0" rpy="0.0 0.0 0.0" />
-            <geometry>
-               <mesh
-                  filename="package://inail2arm_urdf/meshes/simple/mesh_wrist-pitch.stl"
-                  scale="0.001
-               ${rot*0.001} 0.001" />
-            </geometry>
-         </collision> -->
-      </link>
-      <!--wrist-pitch -->
-      <!-- /LINKS -->
-      <!-- JOINTS -->
-      <!-- shoulder yaw -->
-      <joint name="j_arm${arm_num}_1" type="revolute">
-         <parent link="${parent}" />
-         <child link="arm${arm_num}_1" />
-         <axis xyz="0 0 1" />
-         <origin xyz="${Shoulder_1_Ox} ${rot*Shoulder_1_Oy} ${Shoulder_1_Oz}"
-            rpy="${rot*Shoulder_1_roll} ${Shoulder_1_pitch} ${Shoulder_1_yaw}" />
-         <limit lower="${j_arm_1_lower[arm_num-1]}" upper="${j_arm_1_upper[arm_num-1]}"
-            effort="${j_arm_1_torque[arm_num-1]}" velocity="${j_arm_1_velocity[arm_num-1]}" />
-      </joint>
-      <!-- shoulder yaw -->
-      <!-- shoulder pitch -->
-      <joint name="j_arm${arm_num}_2" type="revolute">
-         <parent link="arm${arm_num}_1" />
-         <child link="arm${arm_num}_2" />
-         <origin xyz="${Shoulder_2_Ox} ${rot*Shoulder_2_Oy} ${Shoulder_2_Oz}"
-            rpy="${rot*Shoulder_2_roll} ${Shoulder_2_pitch} ${Shoulder_2_yaw}" />
-         <axis xyz="0 0 -1" />
-         <limit lower="${j_arm_2_lower[arm_num-1]}" upper="${j_arm_2_upper[arm_num-1]}"
-            effort="${j_arm_2_torque[arm_num-1]}" velocity="${j_arm_2_velocity[arm_num-2]}" />
-      </joint>
-      <!-- shoulder pitch -->
-      <!-- elbow yaw -->
-      <joint name="j_arm${arm_num}_3" type="revolute">
-         <parent link="arm${arm_num}_2" />
-         <child link="arm${arm_num}_3" />
-         <origin xyz="${Elbow_1_Ox} ${rot*Elbow_1_Oy} ${Elbow_1_Oz}"
-            rpy="${rot*Elbow_1_roll} ${Elbow_1_pitch} ${Elbow_1_yaw}" />
-         <axis xyz="0 0 1" />
-         <limit lower="${j_arm_3_lower[arm_num-1]}" upper="${j_arm_3_upper[arm_num-1]}"
-            effort="${j_arm_3_torque[arm_num-1]}" velocity="${j_arm_3_velocity[arm_num-1]}" />
-      </joint>
-      <!-- elbow yaw -->
-      <!-- forearm yaw -->
-      <joint name="j_arm${arm_num}_4" type="revolute">
-         <parent link="arm${arm_num}_3" />
-         <child link="arm${arm_num}_4" />
-         <origin xyz="${Forearm_1_Ox} ${Forearm_1_Oy} ${Forearm_1_Oz}"
-            rpy="${rot*Forearm_1_roll} ${Forearm_1_pitch} ${Forearm_1_yaw}" />
-         <axis xyz="0 0 1" />
-         <limit lower="${j_arm_4_lower[arm_num-1]}" upper="${j_arm_4_upper[arm_num-1]}"
-            effort="${j_arm_4_torque[arm_num-1]}" velocity="${j_arm_4_velocity[arm_num-1]}" />
-      </joint>
-      <!-- forearm yaw -->
-      <!-- wrist pitch-->
-      <joint name="j_arm${arm_num}_5" type="revolute">
-         <parent link="arm${arm_num}_4" />
-         <child link="arm${arm_num}_5" />
-         <origin xyz="${Wrist_1_Ox} ${rot*Wrist_1_Oy} ${Wrist_1_Oz}"
-            rpy="${rot*Wrist_1_roll} ${Wrist_1_pitch} ${Wrist_1_yaw}" />
-         <axis xyz="0 0 1" />
-         <limit lower="${j_arm_5_lower[arm_num-1]}" upper="${j_arm_5_upper[arm_num-1]}"
-            effort="${j_arm_5_torque[arm_num-1]}" velocity="${j_arm_5_velocity[arm_num-1]}" />
-      </joint>
-      <!-- wrist pitch-->
-      <!-- wrist2 pitch-->
-      <joint name="j_arm${arm_num}_6" type="revolute">
-         <parent link="arm${arm_num}_5" />
-         <child link="arm${arm_num}_6" />
-         <origin xyz="${Wrist_2_Ox} ${rot*Wrist_2_Oy} ${Wrist_2_Oz}"
-               rpy="${rot*Wrist_2_roll} ${Wrist_2_pitch} ${Wrist_2_yaw}" />
-         <axis xyz="0 0 1" />
-         <limit lower="${j_arm_6_lower[arm_num-1]}" upper="${j_arm_6_upper[arm_num-1]}"
-            effort="${j_arm_6_torque[arm_num-1]}" velocity="${j_arm_6_velocity[arm_num-1]}" />
-      </joint>
-      <!-- /wrist2 pitch-->
-   </xacro:macro>
-   <!-- /macro arms -->
+<robot xmlns:xacro="http://ros.org/wiki/xacro" name="inail2arm">
+    <xacro:include filename="$(find inail2arm_urdf)/urdf/conversions.urdf.xacro" />
+    <xacro:include filename="$(find inail2arm_urdf)/urdf/materials.urdf.xacro" />
+    <xacro:include filename="$(find inail2arm_urdf)/urdf/inail2arm_macro.urdf.xacro" />
+    <xacro:include filename="$(find inail2arm_urdf)/urdf/inail2base.urdf.xacro" />
+    <xacro:include filename="$(find inail2arm_urdf)/urdf/kinematics_properties.urdf.xacro" />
+    <xacro:include filename="$(find inail2arm_urdf)/urdf/inertial_properties.urdf.xacro" />
+    <xacro:include filename="$(find inail2arm_urdf)/urdf/limits.urdf.xacro" />
+    <link name="world"/>
+    <xacro:inail2_base rot="1" parent="world">
+      <origin xyz="0 0 0" rpy="0 0 0"/>
+    </xacro:inail2_base>
+    <xacro:inail2_arm arm_num="1"  rot="1"  parent="base_link">
+      <origin xyz="0 0 0" rpy="0 0 0"/>
+    </xacro:inail2_arm>
 </robot>

File: inail2arm_urdf/urdf/kinematics_properties.urdf.xacro (robot description, xacro)
@@ -38,6 +38,6 @@
 <!-- Origin -->
 <xacro:property name="Wrist_2_Ox" value=" 0.0 "/>
-<xacro:property name="Wrist_2_Oy" value=" -0.0 "/>
-<xacro:property name="Wrist_2_Oz" value=" 0.0 "/>
+<xacro:property name="Wrist_2_Oy" value=" -0.02 "/>
+<xacro:property name="Wrist_2_Oz" value=" 0.043 "/>
 <xacro:property name="Wrist_2_roll" value=" 0"/>
 <xacro:property name="Wrist_2_pitch" value=" 0.0 "/>

File: inail2arm_urdf/urdf/limits.urdf.xacro (robot description, xacro)
@@ -2,16 +2,16 @@
 <robot  xmlns:xacro="http://ros.org/wiki/xacro">
 <!-- Origin -->
-<xacro:property name="j_arm_1_lower" value="${[-3.0]}"/>
-<xacro:property name="j_arm_2_lower" value="${[-3.0]}"/>
-<xacro:property name="j_arm_3_lower" value="${[-3.0]}"/>
-<xacro:property name="j_arm_4_lower" value="${[-3.0]}"/>
-<xacro:property name="j_arm_5_lower" value="${[-3.0]}"/>
-<xacro:property name="j_arm_6_lower" value="${[-3.0]}"/>
-<xacro:property name="j_arm_1_upper" value="${[3.0]}"/>
-<xacro:property name="j_arm_2_upper" value="${[3.0]}"/>
-<xacro:property name="j_arm_3_upper" value="${[3.0]}"/>
-<xacro:property name="j_arm_4_upper" value="${[3.0]}"/>
-<xacro:property name="j_arm_5_upper" value="${[3.0]}"/>
-<xacro:property name="j_arm_6_upper" value="${[3.0]}"/>
+<xacro:property name="j_arm_1_lower" value="${[-2.85]}"/>
+<xacro:property name="j_arm_2_lower" value="${[-2.0]}"/>
+<xacro:property name="j_arm_3_lower" value="${[-2.2]}"/>
+<xacro:property name="j_arm_4_lower" value="${[-2.7]}"/>
+<xacro:property name="j_arm_5_lower" value="${[-2.2]}"/>
+<xacro:property name="j_arm_6_lower" value="${[-2.85]}"/>
+<xacro:property name="j_arm_1_upper" value="${[2.85]}"/>
+<xacro:property name="j_arm_2_upper" value="${[2.0]}"/>
+<xacro:property name="j_arm_3_upper" value="${[2.2]}"/>
+<xacro:property name="j_arm_4_upper" value="${[2.7]}"/>
+<xacro:property name="j_arm_5_upper" value="${[2.2]}"/>
+<xacro:property name="j_arm_6_upper" value="${[2.85]}"/>
 <xacro:property name="j_arm_1_velocity" value="${[3.86, 3.86 ]}"/>
 <xacro:property name="j_arm_2_velocity" value="${[3.86, 3.86 ]}"/>
