Commit message: arm1_6 mesh added

File: inail2arm_srdf/srdf/inail2arm.srdf.xacro (robot description, xacro)
@@ -33,20 +33,27 @@
     <disable_collisions link1="arm1_1" link2="arm1_4" reason="Never"/>
     <disable_collisions link1="arm1_1" link2="arm1_5" reason="Never"/>
+    <disable_collisions link1="arm1_1" link2="arm1_6" reason="Never"/>
     <disable_collisions link1="arm1_1" link2="base_link" reason="Adjacent"/>
     <disable_collisions link1="arm1_2" link2="arm1_3" reason="Adjacent"/>
     <disable_collisions link1="arm1_2" link2="arm1_5" reason="Never"/>
+    <disable_collisions link1="arm1_2" link2="arm1_6" reason="Never"/>
     <disable_collisions link1="arm1_2" link2="base_link" reason="Never"/>
     <disable_collisions link1="arm1_3" link2="arm1_4" reason="Adjacent"/>
     <disable_collisions link1="arm1_3" link2="arm1_5" reason="Never"/>
+    <disable_collisions link1="arm1_3" link2="arm1_6" reason="Never"/>
     <disable_collisions link1="arm1_3" link2="base_link" reason="Never"/>
     <disable_collisions link1="arm1_4" link2="arm1_5" reason="Adjacent"/>
+    <disable_collisions link1="arm1_4" link2="arm1_6" reason="Never"/>
+    <disable_collisions link1="arm1_5" link2="arm1_6" reason="Adjacent"/>
     <xacro:if value="${END_EFFECTOR == 'dagana' or END_EFFECTOR == 'dagana_fixed'}">
         <disable_collisions link1="arm1_3" link2="dagana_1_bottom_link" reason="Never"/>
         <disable_collisions link1="arm1_3" link2="dagana_1_top_link" reason="Never"/>
+        <disable_collisions link1="arm1_4" link2="dagana_1_bottom_link" reason="Never"/>
+        <disable_collisions link1="arm1_4" link2="dagana_1_top_link" reason="Never"/>
         <disable_collisions link1="arm1_5" link2="dagana_1_bottom_link" reason="Never"/>
-        <disable_collisions link1="arm1_5" link2="dagana_1_top_link" reason="Adjacent"/>
+        <disable_collisions link1="arm1_5" link2="dagana_1_top_link" reason="Never"/>
+        <disable_collisions link1="arm1_6" link2="dagana_1_bottom_link" reason="Never"/>
+        <disable_collisions link1="arm1_6" link2="dagana_1_top_link" reason="Adjacent"/>
         <disable_collisions link1="dagana_1_bottom_link" link2="dagana_1_top_link" reason="Adjacent"/>
-        <disable_collisions link1="dagana_1_bottom_link" link2="arm1_4" reason="Never"/>
-        <disable_collisions link1="dagana_1_top_link" link2="arm1_4" reason="Never"/>
     </xacro:if>
 </robot>

File: inail2arm_urdf/urdf/inail2arm_ee_macro.urdf.xacro (robot description, xacro)
@@ -9,5 +9,5 @@
             <parent link="${parent}" />
             <child link="tcp_${arm_num}" />
-            <origin xyz="0 0 0" rpy="0. 0. 0."/>
+            <origin xyz="${EE_mount_Ox} ${EE_mount_Oy} ${EE_mount_Oz}" rpy="${EE_mount_roll} ${EE_mount_pitch} ${EE_mount_yaw}"/>
         </joint>
         <!-- virtual tip pitch-->
@@ -16,6 +16,5 @@
         <xacro:include filename="$(find inail2arm_urdf)/urdf/ball.urdf.xacro" />
         <xacro:ball_end_effector arm_num="1" parent_link="${parent}">
-            <!--  TODO check this origin I put it at "occhio"   -->
-            <origin xyz="0 -0.04 0" rpy="-${PI/2} 0 0."/>
+            <origin xyz="${EE_mount_Ox} ${EE_mount_Oy} ${EE_mount_Oz}" rpy="${EE_mount_roll} ${EE_mount_pitch} ${EE_mount_yaw}"/>
         </xacro:ball_end_effector>
         <!--     to have the same final link as when "none" option is used     -->
@@ -30,6 +29,5 @@
         <xacro:include filename="$(find dagana_urdf)/urdf/dagana_macro.urdf.xacro" />
         <xacro:dagana_gripper name="dagana_${arm_num}" parent_link="${parent}" joint_type="fixed">
-            <!--  TODO check this origin I put it at "occhio"   -->
-            <origin xyz="0 -0.018 0" rpy="${PI/2} 0 0"/>
+            <origin xyz="${EE_mount_Ox} ${EE_mount_Oy} ${EE_mount_Oz}" rpy="${EE_mount_roll} ${EE_mount_pitch} ${EE_mount_yaw}"/>
         </xacro:dagana_gripper>
         <!--     to have the same final link as when "none" option is used     -->
@@ -44,6 +42,5 @@
         <xacro:include filename="$(find dagana_urdf)/urdf/dagana_macro.urdf.xacro" />
         <xacro:dagana_gripper name="dagana_${arm_num}" parent_link="${parent}" joint_type="revolute">
-            <!--  TODO check this origin I put it at "occhio"   -->
-            <origin xyz="0 -0.018 0" rpy="${PI/2} 0 0"/>
+            <origin xyz="${EE_mount_Ox} ${EE_mount_Oy} ${EE_mount_Oz}" rpy="${EE_mount_roll} ${EE_mount_pitch} ${EE_mount_yaw}"/>
         </xacro:dagana_gripper>
         <!--     to have the same final link as when "none" option is used     -->

File: inail2arm_urdf/urdf/inail2arm_macro.urdf.xacro (robot description, xacro)
@@ -139,4 +139,21 @@
                iyy="${Wrist_2_yy}" iyz="${rot*Wrist_2_yz}" izz="${Wrist_2_zz}" />
          </inertial>
+         <visual>
+            <origin xyz="0.0 0.0 0.0" rpy="0.0 0.0 0.0" />
+            <geometry>
+               <mesh
+                  filename="package://inail2arm_urdf/meshes/mesh_wrist-roll.stl"
+                  scale="0.001 ${rot*0.001} 0.001" />
+            </geometry>
+            <material name="blue" />
+         </visual>
+         <collision>
+            <origin xyz="0.0 0.0 0.0" rpy="0.0 0.0 0.0" />
+            <geometry>
+               <mesh
+                  filename="package://inail2arm_urdf/meshes/mesh_wrist-roll.stl"
+                  scale="0.001 ${rot*0.001} 0.001" />
+            </geometry>
+         </collision>
       </link>
       <!--wrist-pitch -->
@@ -204,5 +221,5 @@
          <origin xyz="${Wrist_2_Ox} ${rot*Wrist_2_Oy} ${Wrist_2_Oz}"
             rpy="${rot*Wrist_2_roll} ${Wrist_2_pitch} ${Wrist_2_yaw}" />
-         <axis xyz="0 1 0" />
+         <axis xyz="0 0 1" />
          <limit lower="${j_arm_6_lower[arm_num-1]}" upper="${j_arm_6_upper[arm_num-1]}"
             effort="${j_arm_6_torque[arm_num-1]}" velocity="${j_arm_6_velocity[arm_num-1]}" />

Commit message: using dagana with xbot 2.10

File: inail2arm_srdf/srdf/inail2arm.srdf.xacro (robot description, xacro)
@@ -3,16 +3,19 @@
     <xacro:include filename="$(find inail2arm_urdf)/config/inail2arm.urdf.xacro" />
     <group name="arm">
-        <chain base_link="base_link" tip_link="arm1_6"/>
+        <chain base_link="base_link" tip_link="tcp_1"/>
     </group>
     <xacro:if value="${END_EFFECTOR == 'dagana' or END_EFFECTOR == 'dagana_fixed'}">
         <group name="dagana">
-            <chain base_link="arm1_6" tip_link="tcp_1"/>
+            <chain base_link="arm1_6" tip_link="dagana_1_bottom_link"/>
         </group>
     </xacro:if>
     <group name="chains">
         <group name="arm"/>
+        <xacro:if value="${END_EFFECTOR == 'dagana' or END_EFFECTOR == 'dagana_fixed'}">
+            <group name="dagana"></group>
+        </xacro:if>
     </group>
 <!--    <group_state group="arm" name="home">-->
-    <group_state group="chains" name="home">
+    <group_state group="arm" name="home">
         <joint name="j_arm1_1" value="0.0"/>
         <joint name="j_arm1_2" value="0.45"/>
@@ -21,5 +24,9 @@
         <joint name="j_arm1_5" value="1.1"/>
         <joint name="j_arm1_6" value="0.0"/>
+<!--        <xacro:if value="${END_EFFECTOR == 'dagana'}">
+            <joint name="dagana_1_bottom_link" value="0.0"/>
+        </xacro:if>-->
     </group_state>
+    <!--  For moveit    -->
     <!--END EFFECTOR: Purpose: Represent information about an end effector.-->
     <xacro:if value="${END_EFFECTOR == 'dagana' or END_EFFECTOR == 'dagana_fixed'}">

File: inail2arm_urdf/config/inail2arm.urdf.xacro (robot description, xacro)
@@ -3,9 +3,11 @@
 <xacro:property name="model_name" value="inail2arm" />
 <xacro:property name="model_version" value="0.1" />
-<xacro:arg name="end_effector" default="none"/> <!-- none, ball, dagana_fixed, dagana -->
+<xacro:arg name="end_effector" default="dagana"/> <!-- none, ball, dagana_fixed, dagana -->
 <xacro:property name="END_EFFECTOR" value="$(arg end_effector)" />
 <!-- HACK to add standalone dagana plugin and ignore the dagana joint in the libxbot2_gz_joint_server -->
 <!-- This property is used in the gazebo/xbot.gazebo.xacro file -->
 <!-- In future, xbot will be able to ignore end-effectors in the hal and this should not be neccesary anymore -->
-<xacro:property name="DAGANA_STANDALONE_PLUGIN" value="true" />
+<xacro:property name="DAGANA_STANDALONE_PLUGIN" value="false" />
+<xacro:arg name="proximity_sensors" default="true"/>
+<xacro:property name="PROXIMITY_SENSORS" value="$(arg proximity_sensors)" />
 </robot>

File: inail2arm_urdf/urdf/inail2arm.urdf (robot description, URDF)
Before this commit: robot inail2arm, 18 links, 17 joints
Links:
- added link dagana_1_bottom_link, mass 4.6117745e-01; collision mesh filename=package://dagana_urdf/meshes/dg0002-ch.stl scale=0.001 0.001 0.001; visual mesh filename=package://dagana_urdf/meshes/dg0002.stl scale=0.001 0.001 0.001
- added link dagana_1_tcp
- added link dagana_1_top_link, mass 1.7432400; collision mesh filename=package://dagana_urdf/meshes/dg0001-simplified_v2.stl scale=0.001 0.001 0.001; visual mesh filename=package://dagana_urdf/meshes/dg0001-simplified.stl scale=0.001 0.001 0.001
Joints:
- added joint dagana_1_claw_joint: type revolute, parent dagana_1_top_link, child dagana_1_bottom_link, origin xyz=0.0 -0.028 0.05025 rpy=1.57079632679 0 3.14159265359, axis -1 0 0, limit lower=0 upper=1 effort=1000 velocity=2.0
- added joint dagana_1_mount_joint: type fixed, parent arm1_6, child dagana_1_top_link, origin xyz=0.0 0.0 0.03475 rpy=0.0 0.0 0.0
- added joint dagana_1_tcp_joint: type fixed, parent dagana_1_top_link, child dagana_1_tcp, origin xyz=0 -0.05 0.15 rpy=0 0 0
- joint j_tcp_1: origin xyz=0.0 0.0 0.03475 rpy=0.0 0.0 0.0 -> xyz=0 0 0 rpy=0 0 0; parent arm1_6 -> dagana_1_tcp

Commit message: configs devels

File: inail2arm_srdf/srdf/inail2arm.srdf.xacro (robot description, xacro)
@@ -34,5 +34,5 @@
     </xacro:if>
     <!--VIRTUAL JOINT: Purpose: this element defines a virtual joint between a robot link and an external frame of reference (considered fixed with respect to the robot)-->
-    <virtual_joint name="base_joint" type="fixed" parent_frame="world" child_link="base_link"/>
+    <virtual_joint name="reference" type="fixed" parent_frame="world" child_link="base_link"/>
     <!--DISABLE COLLISIONS: By default it is assumed that any link of the robot could potentially come into collision with any other link in the robot. This tag disables collision checking between a specified pair of links. -->
     <disable_collisions link1="arm1_1" link2="arm1_2" reason="Adjacent"/>

File: inail2arm_urdf/urdf/gazebo/xbot.gazebo.xacro (robot description, xacro)
@@ -26,5 +26,5 @@
         <pid>
             <gain name="lowpwr_mot" p="50"  d="5"/>
-            <gain name="small_mot"  p="800"  d="8"/>
+            <gain name="small_mot"  p="600"  d="6"/>
             <gain name="medium_mot" p="4000" d="40"/>
             <gain name="big_mot"    p="8000" d="50"/>

File: inail2arm_urdf/urdf/inail2arm.urdf.xacro (robot description, xacro)
@@ -8,4 +8,5 @@
     <xacro:arg name="yaw" default="0"/>
     <xacro:arg name="parent" default=""/>
+    <xacro:property name="parent" default="$(arg parent)"/>
     <xacro:include filename="$(find inail2arm_urdf)/config/inail2arm.urdf.xacro" />
     <xacro:include filename="$(find inail2arm_urdf)/urdf/conversions.urdf.xacro" />
@@ -17,5 +18,8 @@
     <xacro:include filename="$(find inail2arm_urdf)/urdf/inertial_properties.urdf.xacro" />
     <xacro:include filename="$(find inail2arm_urdf)/urdf/limits.urdf.xacro" />
-    <xacro:inail2_base rot="1" parent="$(arg parent)">
+    <xacro:unless value="${parent == ''}">
+        <link name="${parent}"/>
+    </xacro:unless>
+    <xacro:inail2_base rot="1" parent="${parent}">
         <origin xyz="$(arg x) $(arg y) $(arg z)" rpy="$(arg roll) $(arg pitch) $(arg yaw)"/>
     </xacro:inail2_base>
