Commit message: updated homing pos, headless gazebo + rviz

File: inail2arm_srdf/srdf/inail2_dual_arm.srdf.xacro (robot description, xacro)
@@ -13,13 +13,13 @@
     </group>
     <group_state group="chains" name="home">
-        <joint name="j_arm2_1" value="1.3"/>
-        <joint name="j_arm2_2" value="0.0"/>
-        <joint name="j_arm2_3" value="1.4"/>
+        <joint name="j_arm2_1" value="-1.7"/>
+        <joint name="j_arm2_2" value="-0.4"/>
+        <joint name="j_arm2_3" value="1.7"/>
         <joint name="j_arm2_4" value="1.4"/>
         <joint name="j_arm2_5" value="1.57"/>
         <joint name="j_arm2_6" value="0.0"/>
-        <joint name="j_arm1_1" value="1.84"/>
-        <joint name="j_arm1_2" value="0.0"/>
-        <joint name="j_arm1_3" value="-1.4"/>
+        <joint name="j_arm1_1" value="1.7"/>
+        <joint name="j_arm1_2" value="0.4"/>
+        <joint name="j_arm1_3" value="-1.7"/>
         <joint name="j_arm1_4" value="-1.4"/>
         <joint name="j_arm1_5" value="-1.57"/>

Commit message: dual arm with dagana tests

File: inail2arm_srdf/srdf/inail2_dual_arm.srdf.xacro (robot description, xacro)
@@ -8,9 +8,30 @@
         <chain base_link="base_link" tip_link="arm2_6"/>
     </group>
+    <group name="dagana_1">
+        <chain base_link="arm1_6" tip_link="dagana_1_bottom_link"/>
+    </group>
+    <group name="dagana_2">
+        <chain base_link="arm2_6" tip_link="dagana_2_bottom_link"/>
+    </group>
     <group name="chains">
         <group name="left_arm"/>
         <group name="right_arm"/>
+        <group name="dagana_1" />
+        <group name="dagana_2" />
     </group>
     <group_state group="chains" name="home">
+        <joint name="j_arm2_1" value="-1.7"/>
+        <joint name="j_arm2_2" value="-0.4"/>
+        <joint name="j_arm2_3" value="1.7"/>
+        <joint name="j_arm2_4" value="0.0"/>
+        <joint name="j_arm2_5" value="-1.25"/>
+        <joint name="j_arm2_6" value="0.0"/>
+        <joint name="j_arm1_1" value="1.7"/>
+        <joint name="j_arm1_2" value="0.4"/>
+        <joint name="j_arm1_3" value="-1.7"/>
+        <joint name="j_arm1_4" value="0.0"/>
+        <joint name="j_arm1_5" value="1.25"/>
+        <joint name="j_arm1_6" value="0.0"/>
+<!--
         <joint name="j_arm2_1" value="-1.7"/>
         <joint name="j_arm2_2" value="-0.4"/>
@@ -24,5 +45,5 @@
         <joint name="j_arm1_4" value="-1.4"/>
         <joint name="j_arm1_5" value="-1.57"/>
-        <joint name="j_arm1_6" value="0.0"/>
+        <joint name="j_arm1_6" value="0.0"/> -->
     </group_state>
    </robot>

File: inail2arm_urdf/urdf/inail2_dual_arm.urdf.xacro (robot description, xacro)
@@ -60,4 +60,5 @@
         <origin xyz="0.065 -0.153361940777 0.221661940777" rpy="${45*toRad} 0 0"/>
     </joint>
+    <!-- arm 1 -->
     <xacro:inail2_arm arm_num="1"  rot="1"  parent="mount_frame_1">
         <origin xyz="0 0 0" rpy="0 0 ${-90*toRad}"/>
@@ -75,7 +76,12 @@
         <origin xyz="0.065 0.153361940777 0.221661940777" rpy="${-45*toRad} 0 0"/>
     </joint>
+    <!-- arm 2 -->
     <xacro:inail2_arm arm_num="2"  rot="1"  parent="mount_frame_2">
         <origin xyz="0 0 0" rpy="0 0 ${-90*toRad}"/>
     </xacro:inail2_arm>
+    <!-- dagana on arm 1 -->
+    <xacro:inail2_arm_ee arm_num="1"  parent="arm1_6" />
+    <!-- dagana on arm 2 -->
+    <xacro:inail2_arm_ee arm_num="2"  parent="arm2_6" />
     <!--- END EFFECTOR  -->
     <!-- <xacro:inail2_arm_ee arm_num="1"  parent="arm1_6">

Commit message: xbot2 support for dual arm system && minor fixes

File: inail2arm_srdf/srdf/inail2_dual_arm.srdf.xacro (robot description, xacro)
@@ -8,28 +8,32 @@
         <chain base_link="base_link" tip_link="arm2_6"/>
     </group>
-    <group name="dagana_1">
-        <chain base_link="arm1_6" tip_link="dagana_1_bottom_link"/>
-    </group>
-    <group name="dagana_2">
-        <chain base_link="arm2_6" tip_link="dagana_2_bottom_link"/>
-    </group>
+    <xacro:if value="${END_EFFECTOR == 'dagana'}">
+        <group name="dagana_1">
+            <chain base_link="arm1_6" tip_link="dagana_1_bottom_link"/>
+        </group>
+        <group name="dagana_2">
+            <chain base_link="arm2_6" tip_link="dagana_2_bottom_link"/>
+        </group>
+    </xacro:if>
     <group name="chains">
         <group name="left_arm"/>
         <group name="right_arm"/>
-        <group name="dagana_1" />
-        <group name="dagana_2" />
+        <xacro:if value="${END_EFFECTOR == 'dagana'}">
+            <group name="dagana_1" />
+            <group name="dagana_2" />
+        </xacro:if>
     </group>
     <group_state group="chains" name="home">
-        <joint name="j_arm2_1" value="-1.7"/>
-        <joint name="j_arm2_2" value="-0.4"/>
-        <joint name="j_arm2_3" value="1.7"/>
-        <joint name="j_arm2_4" value="0.0"/>
-        <joint name="j_arm2_5" value="-1.25"/>
+        <joint name="j_arm2_1" value="-0.7"/>
+        <joint name="j_arm2_2" value="-0.6"/>
+        <joint name="j_arm2_3" value="1.6"/>
+        <joint name="j_arm2_4" value="0.6"/>
+        <joint name="j_arm2_5" value="-1.5"/>
         <joint name="j_arm2_6" value="0.0"/>
-        <joint name="j_arm1_1" value="1.7"/>
-        <joint name="j_arm1_2" value="0.4"/>
-        <joint name="j_arm1_3" value="-1.7"/>
-        <joint name="j_arm1_4" value="0.0"/>
-        <joint name="j_arm1_5" value="1.25"/>
+        <joint name="j_arm1_1" value="0.7"/>
+        <joint name="j_arm1_2" value="0.6"/>
+        <joint name="j_arm1_3" value="-1.6"/>
+        <joint name="j_arm1_4" value="-0.6"/>
+        <joint name="j_arm1_5" value="1.5"/>
         <joint name="j_arm1_6" value="0.0"/>
 <!--

Commit message: updated drill on arm 2

File: inail2arm_srdf/srdf/inail2_dual_arm.srdf.xacro (robot description, xacro)
@@ -16,4 +16,7 @@
         </group>
     </xacro:if>
+    <group name="inail_drill">
+        <chain base_link="arm2_6" tip_link="drill_chuck"/>
+    </group>
     <group name="chains">
         <group name="left_arm"/>
@@ -23,4 +26,5 @@
             <group name="dagana_2" />
         </xacro:if>
+        <group name="inail_drill" />
     </group>
     <group_state group="chains" name="home">

File: inail2arm_urdf/urdf/inail2_dual_arm.urdf.xacro (robot description, xacro)
@@ -62,5 +62,5 @@
     <!-- arm 1 -->
     <xacro:inail2_arm arm_num="1"  rot="1"  parent="mount_frame_1">
-        <origin xyz="0 0 0" rpy="0 0 ${-90*toRad}"/>
+        <origin xyz="0 0 0" rpy="0 0 ${-45*toRad}"/>
     </xacro:inail2_arm>
     <link name="mount_frame_2">
@@ -78,10 +78,23 @@
     <!-- arm 2 -->
     <xacro:inail2_arm arm_num="2"  rot="1"  parent="mount_frame_2">
-        <origin xyz="0 0 0" rpy="0 0 ${-90*toRad}"/>
+        <origin xyz="0 0 0" rpy="0 0 ${-135*toRad}"/>
     </xacro:inail2_arm>
+    <!-- Drill on arm 2 -->
+  <xacro:include filename="$(find inail_drill_urdf)/urdf/inail_drill_macro.urdf.xacro" />
+  <xacro:inail_drill parent_link="arm2_6">
+    <origin xyz="${EE_mount_Ox} ${EE_mount_Oy} ${EE_mount_Oz+0.003}" rpy="${EE_mount_roll} ${EE_mount_pitch} ${EE_mount_yaw}"/>
+  </xacro:inail_drill>
+<!--
+    <joint name="inail_drill_motor" type="continuous">
+        <origin xyz="0 0 0" rpy="0 0 0"/>
+        <parent link="arm2_6"/>
+        <child link="drill_base"/>
+        <limit effort="30" velocity="100.0" />
+        <limit effort="30" velocity="100.0" lower="-5" upper = "5" />
+    </joint> -->
     <!-- dagana on arm 1 -->
-    <xacro:inail2_arm_ee arm_num="1"  parent="arm1_6" />
+    <!-- <xacro:inail2_arm_ee arm_num="1"  parent="arm1_6" /> -->
     <!-- dagana on arm 2 -->
-    <xacro:inail2_arm_ee arm_num="2"  parent="arm2_6" />
+    <!-- <xacro:inail2_arm_ee arm_num="2"  parent="arm2_6" /> -->
     <!--- END EFFECTOR  -->
     <!-- <xacro:inail2_arm_ee arm_num="1"  parent="arm1_6">

File: inail2arm_urdf/urdf/inail2arm_macro.urdf.xacro (robot description, xacro)
@@ -190,4 +190,11 @@
          <limit lower="${j_arm_3_lower[0]}" upper="${j_arm_3_upper[0]}"
             effort="${j_arm_3_torque[0]}" velocity="${j_arm_3_velocity[0]}" />
+      <!-- Virtual limits for elbow joints, so elbow doesnt flip in undesired orientation: better use cartesio config file to set these-->
+        <!-- <xacro:if value="${parent == 'mount_frame_1'}">
+            <limit lower="${j_arm_3_lower[0]}" upper="${-10*toRad}" effort="${j_arm_3_torque[0]}" velocity="${j_arm_3_velocity[0]}" />
+        </xacro:if>
+        <xacro:if value="${parent == 'mount_frame_2'}">
+            <limit lower="${10*toRad}" upper="${j_arm_3_upper[0]}" effort="${j_arm_3_torque[0]}" velocity="${j_arm_3_velocity[0]}" />
+       </xacro:if> -->
       </joint>
       <!-- elbow yaw -->

File: inail2arm_urdf/urdf/kinematics_properties.urdf.xacro (robot description, xacro)
@@ -38,5 +38,5 @@
 <!-- Origin -->
 <xacro:property name="Wrist_2_Ox" value=" 0.0 "/>
-<xacro:property name="Wrist_2_Oy" value=" -0.033 "/>
+<xacro:property name="Wrist_2_Oy" value=" -0.033 "/> <!-- -0.033  -->
 <xacro:property name="Wrist_2_Oz" value=" 0.043 "/>
 <xacro:property name="Wrist_2_roll" value=" ${PI/2}"/>

File: inail2arm_urdf/urdf/limits.urdf.xacro (robot description, xacro)
@@ -7,5 +7,5 @@
 <xacro:property name="j_arm_4_lower" value="${[-2.7]}"/>
 <xacro:property name="j_arm_5_lower" value="${[-2.2]}"/>
-<xacro:property name="j_arm_6_lower" value="${[-2.85]}"/>
+<xacro:property name="j_arm_6_lower" value="${[-2.7]}"/>
 <xacro:property name="j_arm_1_upper" value="${[2.85]}"/>
 <xacro:property name="j_arm_2_upper" value="${[2.0]}"/>
@@ -13,5 +13,5 @@
 <xacro:property name="j_arm_4_upper" value="${[2.7]}"/>
 <xacro:property name="j_arm_5_upper" value="${[2.2]}"/>
-<xacro:property name="j_arm_6_upper" value="${[2.85]}"/>
+<xacro:property name="j_arm_6_upper" value="${[2.7]}"/>
 <xacro:property name="j_arm_1_velocity" value="${[3.86, 3.86 ]}"/>
 <xacro:property name="j_arm_2_velocity" value="${[3.86, 3.86 ]}"/>
